File: design/kicad/sigmidi-foot-controller.kicad_sch (KiCad schematic)
At the start: 44 parts, among them J1 5.5x2.1mm center-negative, J2 Amphenol ACJS-MHDC, SW1 momentary NO, SW10 momentary NO, SW11 20-detent rotary encoder + NO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, SW2 momentary NO, SW3 momentary NO, SW4 momentary NO, SW5 momentary NO, SW6 momentary NO, SW7 momentary NO, SW8 momentary NO, SW9 momentary NO, U1 DFRobot DFR1075 V1.1, U2 Waveshare 24382, U3 Pololu S13V10F5 #4083

Commit message: Update Nano wiring docs and previews
Parts:
- removed U1: DFRobot DFR1075 V1.1, symbol SIGMIDI:DFR1075_Physical
- added R50: 100k, symbol Device:R
- added R51: 150k, symbol Device:R
- added U1: Arduino Nano ESP32 ABX00083, symbol SIGMIDI:Arduino_Nano_ESP32_Physical
Connections:
- net +9V: now also U1.JP1:15 (VIN/VIN)
- net 3V3: now also U1.JP1:2 (3V3/3V3)
- net ENC_A: now also U1.JP2:7 (D4/GPIO7)
- net ENC_B: now also U1.JP2:8 (D5/GPIO8)
- net ENC_SW: now also U1.JP2:9 (D6/GPIO9)
- net GND: now also R51.2, U1.JP1:14 (GND/GND), U1.JP2:4 (GND/GND)
- net LADDER: now also U1.JP1:4 (A0/GPIO1)
- net LCD_CLK: now also U1.JP2:11 (D8/GPIO17)
- net LCD_CS: now also U1.JP2:13 (D10/GPIO21)
- net LCD_DC: now also U1.JP2:12 (D9/GPIO18)
- net LCD_DIN: now also U1.JP2:14 (D11/GPIO38)
- net LCD_RST: now also U1.JP2:15 (D12/GPIO47)
- net LED_GPIO: now also U1.JP2:10 (D7/GPIO10)
- net P1_ADC: now also U1.JP1:5 (A1/GPIO2)
- net P1_MODE: now also U1.JP2:5 (D2/GPIO5)
- net P2_ADC: now also U1.JP1:7 (A3/GPIO4)
- net P2_MODE: now also U1.JP2:6 (D3/GPIO6)
- new net USB_SENSE: R50.2, R51.1, U1.JP1:8 (A4/GPIO11)
- new net USB_VBUS: R50.1, U1.JP1:12 (VBUS/VUSB/VBUS)
- no-connect marks 21 -> 18
Other:
- note added: "+"
- note added: "+5V LED"
- note added: "0-10k per input. Bias HIGH in resistor mode;"
- note added: "1 BL"
- note added: "1/2/3/7/8/9: NC; pad 13: mechanical / NC"
- note added: "100k"
- note added: "150k"
- note added: "2 RST"
- note added: "20 detents + click"
- note added: "3 D/C"
- note added: "3V3 / Nano logic supply"
- note added: "4 CS"
- note added: "5 SCL / CLK"
- note added: "6 SDA / DIN"
- note added: "7 GND"
- note added: "8 VCC"
- note added: "A0"
- note added: "A1"
- note added: "A2"
- note added: "A3"
- note added: "A4"
- note added: "A5"
- note added: "A6"
- note added: "A7"
- note added: "All printed labels retained; unused pads left unwired."
- note added: "B0"
- note added: "B1"
- note added: "COMMON GND"
- note added: "Check 3.3V data acceptance on the actual LED batch."
- note added: "Component-side top view / USB-C up"
- note added: "Continuous wires connect every fitted terminal. Dots = junctions; crossings without dots = no connection. Component placement is schematic."
- note added: "D0 / RX0"
- note added: "D1 / TX0"
- note added: "D10"
- note added: "D11"
- note added: "D12"
- note added: "D13"
- note added: "D2"
- note added: "D3"
- note added: "D4"
- note added: "D5"
- note added: "D6"
- note added: "D7"
- note added: "D8"
- note added: "D9"
- note added: "J2 ACJS-MHDC / passive pedals"
- note added: "JP1:1"
- note added: "JP1:10"
- note added: "JP1:11"
- note added: "JP1:12 / VBUS"
- note added: "JP1:13"
- note added: "JP1:14 / GND"
- note added: "JP1:15 / VIN"
- note added: "JP1:2 / 3V3"
- note added: "JP1:3"
- note added: "JP1:4 / GPIO1"
- note added: "JP1:5 / GPIO2"
- note added: "JP1:6"
- note added: "JP1:7 / GPIO4"
- note added: "JP1:8 / GPIO11"
- note added: "JP1:9"
- note added: "JP2:1"
- note added: "JP2:10 / GPIO10"
- note added: "JP2:11 / GPIO17"
- note added: "JP2:12 / GPIO18"
- note added: "JP2:13 / GPIO21"
- note added: "JP2:14 / GPIO38"
- note added: "JP2:15 / GPIO47"
- note added: "JP2:2"
- note added: "JP2:3"
- note added: "JP2:4 / GND"
- note added: "JP2:5 / GPIO5"
- note added: "JP2:6 / GPIO6"
- note added: "JP2:7 / GPIO7"
- note added: "JP2:8 / GPIO8"
- note added: "JP2:9 / GPIO9"
- note added: "Lens left, leads right, flat side down."
- note added: "Nano and LCD pins keep physical order. Nano: JP1 left 1-15, JP2 right 15-1, USB-C up. Outlines are schematic."
- note added: "Native USB-C carries USB MIDI and ROM flashing."
- note added: "Netlist, BOM and pin references: design/electrical/. All 46 components and 41 nets checked against the connected drawing."
- note added: "Only LEDs and wires; direct D7 / GPIO10 data."
- note added: "P2 / GH1.25 / SPI / pins 1-8"
- note added: "Pololu 2535 / optional LEDs"
- note added: "Pot: outer legs RING / SLEEVE; wiper TIP."
- note added: "R50"
- note added: "R51"
- note added: "SW11 contact pin arrangement is functional."
- note added: "Set 4 / 6 / 8 / 10 switches; calibrate installed taps."
- note added: "Top to bottom: DIN / 5V / GND / DOUT."
- note added: "U1 Arduino Nano ESP32"
- note added: "USB VBUS sense / 3.0V at 5V"
- note added: "USB-C / MIDI"
- note added: "VBUS / VUSB"
- note added: "Variable resistor: TIP to SLEEVE; RING unused."
- note added: "high impedance in pot / disabled / boot states."
- note added: "v0.1 / KICAD ELECTRICAL SCHEMATIC / external board pins only"
- note removed: "0-10k per input. Bias HIGH in resistor mode; high impedance in pot / disabled / boot."
- note removed: "1.69 inch ST7789V2 / SPI"
- note removed: "1/2/3/7/8/9 NC; 13 mechanical"
- note removed: "1/D6"
- note removed: "14/D3"
- note removed: "15/D13"
- note removed: "16/TX"
- note removed: "17/RX"
- note removed: "18/D7"
- note removed: "19/SDA"
- note removed: "2/A1"
- note removed: "20 detents / NO click"
- note removed: "20/SCL"
- note removed: "21/MI"
- note removed: "22/MO"
- note removed: "23/SCK"
- note removed: "3/A2"
- note removed: "4/A3/LP_RX"
- note removed: "5/A4/LP_TX"
- note removed: "6/D12/LP_SDA"
- note removed: "7/D11/LP_SCL"
- note removed: "8-pin external connector / GH1.25"
- note removed: "8/D2"
- note removed: "9/D9"
- note removed: "All board labels retained; unused pads marked X."
- note removed: "DFRobot and display pins retain physical order. Dots join wires; crossings without dots do not join."
- note removed: "Direct GPIO16 data; check 3.3V acceptance on the actual LED batch."
- note removed: "Dual TRS socket"
- note removed: "J2 ACJS-MHDC"
- note removed: "Lens left / flat down / leads right: DIN, 5V, GND, DOUT."
- note removed: "Module boxes show external terminals only. Layout is schematic; physical footprints are not assigned."
- note removed: "OPTIONAL Pololu 2535 LED CHAIN"
- note removed: "P1:1 / VCC"
- note removed: "P1:10"
- note removed: "P1:11"
- note removed: "P1:12 / GPIO6"
- note removed: "P1:13 / GPIO7"
- note removed: "P1:14"
- note removed: "P1:2 / 3V3"
- note removed: "P1:3 / GND"
- note removed: "P1:4 / GPIO20"
- note removed: "P1:5"
- note removed: "P1:6"
- note removed: "P1:7"
- note removed: "P1:8 / GPIO3"
- note removed: "P1:9 / GPIO2"
- note removed: "P2:1"
- note removed: "P2:1 BL"
- note removed: "P2:10 / GPIO19"
- note removed: "P2:11"
- note removed: "P2:12 / GPIO18"
- note removed: "P2:13 / GPIO1"
- note removed: "P2:14"
- note removed: "P2:15 / GPIO14"
- note removed: "P2:16"
- note removed: "P2:17 / GPIO16"
- note removed: "P2:18 / GPIO17"
- note removed: "P2:2 / 3V3"
- note removed: "P2:2 RST"
- note removed: "P2:3"
- note removed: "P2:3 D/C"
- note removed: "P2:4 / GND"
- note removed: "P2:4 CS"
- note removed: "P2:5"
- note removed: "P2:5 SCL / CLK"
- note removed: "P2:6 / GPIO23"
- note removed: "P2:6 SDA / DIN"
- note removed: "P2:7 / GPIO22"
- note removed: "P2:7 GND"
- note removed: "P2:8 / GPIO21"
- note removed: "P2:8 VCC"
- note removed: "P2:9"
- note removed: "Physical P2 connector: 1 at top"
- note removed: "Pot: outer legs RING / SLEEVE; wiper TIP. Variable resistor: TIP to SLEEVE; RING unused."
- note removed: "SCL"
- note removed: "SDA"
- note removed: "SW1 / click"
- note removed: "Select 4 / 6 / 8 / 10 switches and calibrate fitted taps. SW11 uses functional pin names; verify chosen encoder terminal order."
- note removed: "Top view / USB-C up"
- note removed: "U1 DFRobot DFR1075 V1.1"
- note removed: "v0.1 / KiCad electrical schematic / external board pins only"
